Commit message: forward kinematics and gazebo SCARA

File: urdf/scara.urdf (robot description, URDF)
Before this commit: robot scara, 8 links, 7 joints
Joints:
- joint base_link_to_link_1_v: limit (none) -> effort=100.0 velocity=0.5
- joint joint_2_to_link_3: limit lower=0 upper=1 effort=1000.0 velocity=0.5 -> lower=0 upper=1 effort=100.0 velocity=0.1
- joint link_1_h_to_joint_1: limit (none) -> effort=100.0 velocity=0.5
