Commit message: updated fk and ik node

File: custom_robot_description/urdf/custom_scara.urdf (robot description, URDF)
Before this commit: robot custom_scara, 8 links, 7 joints
Joints:
- joint joint3: limit lower=-1 upper=1 effort=100.0 velocity=0.1 -> lower=-1 upper=1 effort=100.0 velocity=0.5

Commit message: updated ik node

File: custom_robot_description/urdf/custom_scara.urdf (robot description, URDF)
Before this commit: robot custom_scara, 8 links, 7 joints
Joints:
- joint joint3: limit lower=-1 upper=1 effort=100.0 velocity=0.5 -> lower=-1 upper=0.4 effort=100.0 velocity=0.5

Commit message: ref position service

File: custom_robot_description/urdf/custom_scara.urdf (robot description, URDF)
Before this commit: robot custom_scara, 8 links, 7 joints
Joints:
- joint joint3: limit lower=-1 upper=0.4 effort=100.0 velocity=0.5 -> lower=0 upper=1 effort=100.0 velocity=0.5

Commit message: fixed first and second joints

File: custom_robot_description/urdf/custom_scara.urdf (robot description, URDF)
Before this commit: robot custom_scara, 8 links, 7 joints
Joints:
- joint joint1: limit effort=100.0 velocity=0.5 -> (none); type continuous -> fixed
- joint joint2: limit effort=100.0 velocity=0.1 -> (none); type continuous -> fixed

Commit message: joint1 joint2 control

File: custom_robot_description/urdf/custom_scara.urdf (robot description, URDF)
Before this commit: robot custom_scara, 8 links, 7 joints
Joints:
- joint joint1: type fixed -> continuous
- joint joint2: type fixed -> continuous
